File: xmega breakout.brd (EAGLE design)
At the start: 160 x 100 mm, 17 parts, among them IC1 XMEGA16A4A

Commit message: typo
Parts:
- added D1, D2, D3, D4, D5: (no value), fab:SOD123
- C4: value 10uF -> 4.7nF
- R3: value (none) -> 1M
- moved C4 14.6 mm to (44.8, 38.9), turned to 180 degrees
- moved R3 13.6 mm to (45.0, 36.2), turned to 0 degrees
Connections:
- net D+: now also D2.ANODE, D3.CATHODE
- net D-: now also D1.ANODE, D4.CATHODE
- net N$25: now also D3.ANODE, D4.ANODE, D5.ANODE
- net VBUS: now also D1.CATHODE, D2.CATHODE, D5.CATHODE
Changed lines of the file:
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@@
 <element name="R2" library="fab" package="R1206FAB" value="" x="47.578021875" y="43.2023375"/>
 <element name="LED1" library="adafruit" package="1206" value="" x="43.624790625" y="43.318625" rot="R90"/>
-<element name="C4" library="fab" package="C1206" value="10uF" x="40.147890625" y="25.026828125" rot="R90"/>
-<element name="R3" library="fab" package="R1206FAB" value="" x="37.50080625" y="24.892109375" rot="R270"/>
+<element name="C4" library="fab" package="C1206" value="4.7nF" x="44.823171875" y="38.877890625" rot="R180"/>
+<element name="R3" library="fab" package="R1206FAB" value="1M" x="44.957890625" y="36.23080625"/>
 <element name="JP5" library="SparkFun" package="1X08_SMD_ALT" value="" x="49.53" y="62.23" rot="R180"/>
 <element name="JP1" library="SparkFun" package="1X08_SMD_ALT_2X1X4" value="" x="90.214675" y="62.23" rot="R180"/>
+<element name="D1" library="fab" package="SOD123" value="" x="3.81" y="-3.81"/>
+<element name="D2" library="fab" package="SOD123" value="" x="3.81" y="-8.89"/>
+<element name="D3" library="fab" package="SOD123" value="" x="3.81" y="-13.97"/>
+<element name="D4" library="fab" package="SOD123" value="" x="3.81" y="-19.05"/>
+<element name="D5" library="fab" package="SOD123" value="" x="3.81" y="-24.13"/>
 </elements>
 <signals>
@@
 <wire x1="49.76418125" y1="47.795684375" x2="49.76418125" y2="43.737496875" width="0.6096" layer="1"/>
 <wire x1="49.76418125" y1="43.737496875" x2="49.229021875" y2="43.2023375" width="0.6096" layer="1"/>
+<contactref element="D1" pad="CATHODE"/>
+<contactref element="D2" pad="CATHODE"/>
+<contactref element="D5" pad="CATHODE"/>
 <wire x1="49.76418125" y1="43.737496875" x2="96.341234375" y2="28.42404375" width="0" layer="19" extent="1-1"/>
+<wire x1="2.11" y1="-3.81" x2="49.229021875" y2="43.2023375" width="0" layer="19" extent="1-1"/>
+<wire x1="2.11" y1="-8.89" x2="2.11" y2="-3.81" width="0" layer="19" extent="1-1"/>
+<wire x1="2.11" y1="-24.13" x2="2.11" y2="-8.89" width="0" layer="19" extent="1-1"/>
 </signal>
 <signal name="D+">
@@
 <wire x1="87.623634375" y1="26.451715625" x2="87.623634375" y2="23.246365625" width="0.6096" layer="1"/>
 <wire x1="87.623634375" y1="23.246365625" x2="87.63" y2="23.24" width="0.6096" layer="1"/>
+<contactref element="D2" pad="ANODE"/>
+<contactref element="D3" pad="CATHODE"/>
 <wire x1="87.623634375" y1="26.451715625" x2="96.341234375" y2="30.02404375" width="0" layer="19" extent="1-1"/>
+<wire x1="5.51" y1="-8.89" x2="76.769846875" y2="39.217409375" width="0" layer="19" extent="1-1"/>
+<wire x1="2.11" y1="-13.97" x2="5.51" y2="-8.89" width="0" layer="19" extent="1-1"/>
 </signal>
 <signal name="GND">
@@
 <wire x1="53.7401125" y1="42.42640625" x2="59.396965625" y2="37.3352375" width="0.6096" layer="16"/>
 <wire x1="88.007790625" y1="43.538278125" x2="96.341234375" y2="31.62404375" width="0" layer="19" extent="1-1"/>
-<wire x1="40.147890625" y1="26.426828125" x2="43.624790625" y2="44.740625" width="0" layer="19" extent="1-1"/>
-<wire x1="37.50080625" y1="26.543109375" x2="40.147890625" y2="26.426828125" width="0" layer="19" extent="1-1"/>
+<wire x1="43.423171875" y1="38.877890625" x2="43.624790625" y2="44.740625" width="0" layer="19" extent="1-1"/>
+<wire x1="43.306890625" y1="36.23080625" x2="43.423171875" y2="38.877890625" width="0" layer="19" extent="1-1"/>
 </signal>
 <signal name="VCC">
@@
 <wire x1="90.166278125" y1="25.65435625" x2="90.166278125" y2="19.943721875" width="0.6096" layer="1"/>
 <wire x1="90.166278125" y1="19.943721875" x2="90.17" y2="19.94" width="0.6096" layer="1"/>
+<contactref element="D1" pad="ANODE"/>
+<contactref element="D4" pad="CATHODE"/>
 <wire x1="90.166278125" y1="25.65435625" x2="96.341234375" y2="29.22404375" width="0" layer="19" extent="1-1"/>
+<wire x1="5.51" y1="-3.81" x2="77.33553125" y2="39.761346875" width="0" layer="19" extent="1-1"/>
+<wire x1="2.11" y1="-19.05" x2="5.51" y2="-3.81" width="0" layer="19" extent="1-1"/>
 </signal>
 <signal name="N$25">
@@
 <contactref element="C4" pad="1"/>
 <contactref element="U$1" pad="SHIELD@2"/>
+<contactref element="D3" pad="ANODE"/>
+<contactref element="D4" pad="ANODE"/>
+<contactref element="D5" pad="ANODE"/>
 <wire x1="96.341234375" y1="34.52404375" x2="101.841234375" y2="34.52404375" width="0" layer="19" extent="1-1"/>
 <wire x1="101.841234375" y1="25.52404375" x2="101.841234375" y2="34.52404375" width="0" layer="19" extent="1-1"/>
 <wire x1="96.341234375" y1="25.52404375" x2="101.841234375" y2="25.52404375" width="0" layer="19" extent="1-1"/>
-<wire x1="40.147890625" y1="23.626828125" x2="96.341234375" y2="25.52404375" width="0" layer="19" extent="1-1"/>
-<wire x1="37.50080625" y1="23.241109375" x2="40.147890625" y2="23.626828125" width="0" layer="19" extent="1-1"/>
+<wire x1="46.608890625" y1="36.23080625" x2="96.341234375" y2="34.52404375" width="0" layer="19" extent="1-1"/>
+<wire x1="46.223171875" y1="38.877890625" x2="46.608890625" y2="36.23080625" width="0" layer="19" extent="1-1"/>
+<wire x1="5.51" y1="-13.97" x2="46.608890625" y2="36.23080625" width="0" layer="19" extent="1-1"/>
+<wire x1="5.51" y1="-19.05" x2="5.51" y2="-13.97" width="0" layer="19" extent="1-1"/>
+<wire x1="5.51" y1="-24.13" x2="5.51" y2="-19.05" width="0" layer="19" extent="1-1"/>
 </signal>
 <signal name="MISO">
