File: XMEGAbreakoutSMD.sch (EAGLE design)
At the start: 24 parts, among them IC1 XMEGA16A4

Commit message: fix to smd board
Parts:
- removed C3: 0.1uF, fab:CAP-US1206
- removed JUMPER2: 0, fab:RES-US1206FAB
Connections:
- net GND: no longer C3.2
- net RESET: no longer C3.1
- net VCC: now also JP6.2
Changed lines of the file:
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@@
 <?xml version="1.0" encoding="utf-8"?>
 <!DOCTYPE eagle SYSTEM "eagle.dtd">
-<eagle version="7.1.0">
+<eagle version="7.5.0">
 <drawing>
 <settings>
@@
 <grid distance="0.1" unitdist="inch" unit="inch" style="lines" multiple="1" display="no" altdistance="0.01" altunitdist="inch" altunit="inch"/>
 <layers>
-<layer number="1" name="Top" color="4" fill="1" visible="yes" active="no"/>
-<layer number="2" name="Route2" color="1" fill="3" visible="yes" active="no"/>
-<layer number="3" name="Route3" color="4" fill="3" visible="yes" active="no"/>
-<layer number="14" name="Route14" color="1" fill="6" visible="yes" active="no"/>
-<layer number="15" name="Route15" color="4" fill="6" visible="yes" active="no"/>
-<layer number="16" name="Bottom" color="1" fill="1" visible="yes" active="no"/>
-<layer number="17" name="Pads" color="2" fill="1" visible="yes" active="no"/>
-<layer number="18" name="Vias" color="2" fill="1" visible="yes" active="no"/>
-<layer number="19" name="Unrouted" color="6" fill="1" visible="yes" active="no"/>
-<layer number="20" name="Dimension" color="15" fill="1" visible="yes" active="no"/>
-<layer number="21" name="tPlace" color="7" fill="1" visible="yes" active="no"/>
-<layer number="22" name="bPlace" color="7" fill="1" visible="yes" active="no"/>
-<layer number="23" name="tOrigins" color="15" fill="1" visible="yes" active="no"/>
-<layer number="24" name="bOrigins" color="15" fill="1" visible="yes" active="no"/>
-<layer number="25" name="tNames" color="7" fill="1" visible="yes" active="no"/>
-<layer number="26" name="bNames" color="7" fill="1" visible="yes" active="no"/>
-<layer number="27" name="tValues" color="7" fill="1" visible="yes" active="no"/>
-<layer number="28" name="bValues" color="7" fill="1" visible="yes" active="no"/>
+<layer number="1" name="Top" color="4" fill="1" visible="no" active="no"/>
+<layer number="2" name="Route2" color="1" fill="3" visible="no" active="no"/>
+<layer number="3" name="Route3" color="4" fill="3" visible="no" active="no"/>
+<layer number="14" name="Route14" color="1" fill="6" visible="no" active="no"/>
+<layer number="15" name="Route15" color="4" fill="6" visible="no" active="no"/>
+<layer number="16" name="Bottom" color="1" fill="1" visible="no" active="no"/>
+<layer number="17" name="Pads" color="2" fill="1" visible="no" active="no"/>
+<layer number="18" name="Vias" color="2" fill="1" visible="no" active="no"/>
+<layer number="19" name="Unrouted" color="6" fill="1" visible="no" active="no"/>
+<layer number="20" name="Dimension" color="15" fill="1" visible="no" active="no"/>
+<layer number="21" name="tPlace" color="7" fill="1" visible="no" active="no"/>
+<layer number="22" name="bPlace" color="7" fill="1" visible="no" active="no"/>
+<layer number="23" name="tOrigins" color="15" fill="1" visible="no" active="no"/>
+<layer number="24" name="bOrigins" color="15" fill="1" visible="no" active="no"/>
+<layer number="25" name="tNames" color="7" fill="1" visible="no" active="no"/>
+<layer number="26" name="bNames" color="7" fill="1" visible="no" active="no"/>
+<layer number="27" name="tValues" color="7" fill="1" visible="no" active="no"/>
+<layer number="28" name="bValues" color="7" fill="1" visible="no" active="no"/>
 <layer number="29" name="tStop" color="7" fill="3" visible="no" active="no"/>
 <layer number="30" name="bStop" color="7" fill="6" visible="no" active="no"/>
@@
 <layer number="35" name="tGlue" color="7" fill="4" visible="no" active="no"/>
 <layer number="36" name="bGlue" color="7" fill="5" visible="no" active="no"/>
-<layer number="37" name="tTest" color="7" fill="1" visible="yes" active="no"/>
-<layer number="38" name="bTest" color="7" fill="1" visible="yes" active="no"/>
+<layer number="37" name="tTest" color="7" fill="1" visible="no" active="no"/>
+<layer number="38" name="bTest" color="7" fill="1" visible="no" active="no"/>
 <layer number="39" name="tKeepout" color="4" fill="11" visible="no" active="no"/>
 <layer number="40" name="bKeepout" color="1" fill="11" visible="no" active="no"/>
@@
 <layer number="44" name="Drills" color="7" fill="1" visible="no" active="no"/>
 <layer number="45" name="Holes" color="7" fill="1" visible="no" active="no"/>
-<layer number="46" name="Milling" color="3" fill="1" visible="yes" active="no"/>
-<layer number="47" name="Measures" color="7" fill="1" visible="yes" active="no"/>
-<layer number="48" name="Document" color="7" fill="1" visible="yes" active="no"/>
-<layer number="49" name="Reference" color="7" fill="1" visible="yes" active="no"/>
-<layer number="50" name="dxf" color="7" fill="1" visible="yes" active="no"/>
-<layer number="51" name="tDocu" color="7" fill="1" visible="yes" active="no"/>
-<layer number="52" name="bDocu" color="7" fill="1" visible="yes" active="no"/>
-<layer number="53" name="tGND_GNDA" color="7" fill="9" visible="yes" active="no"/>
-<layer number="54" name="bGND_GNDA" color="1" fill="9" visible="yes" active="no"/>
-<layer number="56" name="wert" color="7" fill="1" visible="yes" active="no"/>
+<layer number="46" name="Milling" color="3" fill="1" visible="no" active="no"/>
+<layer number="47" name="Measures" color="7" fill="1" visible="no" active="no"/>
+<layer number="48" name="Document" color="7" fill="1" visible="no" active="no"/>
+<layer number="49" name="Reference" color="7" fill="1" visible="no" active="no"/>
+<layer number="50" name="dxf" color="7" fill="1" visible="no" active="no"/>
+<layer number="51" name="tDocu" color="7" fill="1" visible="no" active="no"/>
+<layer number="52" name="bDocu" color="7" fill="1" visible="no" active="no"/>
+<layer number="53" name="tGND_GNDA" color="7" fill="9" visible="no" active="no"/>
+<layer number="54" name="bGND_GNDA" color="1" fill="9" visible="no" active="no"/>
+<layer number="56" name="wert" color="7" fill="1" visible="no" active="no"/>
 <layer number="90" name="Modules" color="5" fill="1" visible="yes" active="yes"/>
 <layer number="91" name="Nets" color="2" fill="1" visible="yes" active="yes"/>
@@
 <part name="R1" library="fab" deviceset="RES-US" device="1206FAB" value="10K"/>
 <part name="S1" library="fab" deviceset="6MM_SWITCH" device="6MM_SWITCH"/>
-<part name="C3" library="fab" deviceset="CAP-US" device="1206" value="0.1uF"/>
 <part name="U$1" library="fab" deviceset="USB_MINIB" device=""/>
 <part name="JP4" library="fab" deviceset="PINHD-2X3-SMD" device=""/>
@@
 <part name="GND5" library="SparkFun" deviceset="GND" device=""/>
 <part name="JUMPER1" library="fab" deviceset="RES-US" device="1206FAB" value="0"/>
-<part name="JUMPER2" library="fab" deviceset="RES-US" device="1206FAB" value="0"/>
 <part name="C5" library="fab" deviceset="CAP-US" device="1206" value="4.7uF"/>
 <part name="U$2" library="SparkFun" deviceset="INVERTER" device=""/>
@@
 <part name="JP6" library="fab" deviceset="PINHD-2X3-SMD" device=""/>
 <part name="GND6" library="SparkFun" deviceset="GND" device=""/>
+<part name="P+2" library="SparkFun" deviceset="VCC" device=""/>
 </parts>
 <sheets>
@@
 <instance part="R1" gate="G$1" x="-25.4" y="93.98" rot="R180"/>
 <instance part="S1" gate="2" x="-48.26" y="93.98" rot="R270"/>
-<instance part="C3" gate="G$1" x="-48.26" y="76.2" rot="R180"/>
 <instance part="U$1" gate="G$1" x="-63.5" y="154.94" rot="R180"/>
 <instance part="JP4" gate="A" x="139.7" y="48.26"/>
@@
 <instance part="GND5" gate="1" x="106.68" y="142.24"/>
 <instance part="JUMPER1" gate="G$1" x="0" y="175.26"/>
-<instance part="JUMPER2" gate="G$1" x="0" y="167.64"/>
 <instance part="C5" gate="G$1" x="30.48" y="162.56" rot="R270"/>
 <instance part="U$2" gate="G$1" x="30.48" y="116.84"/>
@@
 <instance part="JP6" gate="A" x="139.7" y="20.32"/>
 <instance part="GND6" gate="1" x="157.48" y="12.7"/>
+<instance part="P+2" gate="1" x="157.48" y="25.4"/>
 </instances>
 <busses>
@@
 <wire x1="-43.18" y1="93.98" x2="-43.18" y2="91.44" width="0.1524" layer="91"/>
 <junction x="-43.18" y="93.98"/>
-<pinref part="C3" gate="G$1" pin="1"/>
-<wire x1="-45.72" y1="76.2" x2="-35.56" y2="76.2" width="0.1524" layer="91"/>
-<wire x1="-35.56" y1="76.2" x2="-35.56" y2="93.98" width="0.1524" layer="91"/>
 <junction x="-35.56" y="93.98"/>
 <wire x1="-35.56" y1="93.98" x2="-35.56" y2="106.68" width="0.1524" layer="91"/>
@@
 <pinref part="S1" gate="2" pin="P1"/>
 <wire x1="-53.34" y1="93.98" x2="-53.34" y2="91.44" width="0.1524" layer="91"/>
-<wire x1="-53.34" y1="93.98" x2="-60.96" y2="93.98" width="0.1524" layer="91"/>
 <junction x="-53.34" y="93.98"/>
-<pinref part="C3" gate="G$1" pin="2"/>
-<wire x1="-53.34" y1="76.2" x2="-60.96" y2="76.2" width="0.1524" layer="91"/>
-<wire x1="-60.96" y1="76.2" x2="-60.96" y2="93.98" width="0.1524" layer="91"/>
 <pinref part="GND4" gate="1" pin="GND"/>
-<wire x1="-60.96" y1="93.98" x2="-73.66" y2="93.98" width="0.1524" layer="91"/>
+<wire x1="-53.34" y1="93.98" x2="-73.66" y2="93.98" width="0.1524" layer="91"/>
 <wire x1="-73.66" y1="93.98" x2="-73.66" y2="91.44" width="0.1524" layer="91"/>
-<junction x="-60.96" y="93.98"/>
 </segment>
 <segment>
@@
 <label x="144.78" y="162.56" size="1.778" layer="95"/>
 </segment>
-</net>
+<segment>
+<pinref part="JP6" gate="A" pin="2"/>
+<wire x1="144.78" y1="22.86" x2="157.48" y2="22.86" width="0.1524" layer="91"/>
+<pinref part="P+2" gate="1" pin="VCC"/>
+<wire x1="157.48" y1="25.4" x2="157.48" y2="22.86" width="0.1524" layer="91"/>
+</segment>
+</net>
