File: XMEGAbreakoutTH.brd (EAGLE design)
At the start: 160 x 100 mm, 24 parts, among them IC1 XMEGA16A4

Commit message: eagle layout finished
Parts:
- JP1: device SparkFun:1X08_SMD_ALT_2X1X4 -> SparkFun:1X08_2X1X4
- JP2, JP3, JP5: device SparkFun:1X08_SMD_ALT -> SparkFun:1X08
- moved JP1 20.4 mm to (69.8, 62.2), turned to 0 degrees
- turned JP2 to 180 degrees
- turned JP3 to 180 degrees
- turned JP5 to 0 degrees
Routing:
- net PA4: track 13.7 -> 17.0 mm
- net PE0: track 46.0 -> 47.7 mm
- net PA7: track 21.8 -> 20.2 mm
- net PE3: track 44.2 -> 42.6 mm
- net N$13: track 34.6 -> 33.0 mm
- net SCK: track 28.7 -> 27.0 mm
- net PA5: track 17.1 -> 15.4 mm
- net N$9: track 30.3 -> 28.7 mm
- net N$11: track 25.9 -> 24.3 mm
- net N$24: track 17.4 -> 19.0 mm
- net N$23: track 20.9 -> 19.2 mm
- net N$21: track 19.3 -> 17.7 mm
- net N$19: track 22.1 -> 20.4 mm
- net N$15: track 37.6 -> 35.9 mm
- net N$12: track 30.2 -> 31.9 mm
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
Commit message: final designs
Parts:
- moved C2 17.6 mm to (58.3, 47.1)
- moved C1 11.6 mm to (53.7, 47.8), turned to 270 degrees
Connections:
- net GND: now also IC2.1; no longer IC2.2
- net VBUS: now also IC2.3; no longer IC2.1
- net VCC: now also IC2.2; no longer IC2.3
Routing:
- net VBUS: track 99.6 -> 107.4 mm
- net VCC: track 61.3 -> 55.9 mm
- net GND: track 158.3 -> 163.4 mm, vias 8 -> 9
- net RESET: track 182.6 -> 179.9 mm

Commit message: small changes
Parts:
- added C5: 4.7uF, fab:C1206
Connections:
- net GND: now also C5.2
- net VBUS: now also C5.1
Routing:
- net VBUS: track 107.4 -> 110.9 mm
- net GND: track 163.4 -> 165.4 mm
Changed lines of the file:
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@@
 <element name="JUMPER1" library="fab" package="R1206FAB" value="0" x="86.0425" y="31.4325" rot="R220"/>
 <element name="JUMPER2" library="fab" package="R1206FAB" value="0" x="69.85" y="18.0975" rot="R90"/>
+<element name="C5" library="fab" package="C1206" value="4.7uF" x="46.99" y="54.61" rot="R180"/>
 </elements>
 <signals>
@@
 <wire x1="49.76418125" y1="52.395684375" x2="47.950684375" y2="52.395684375" width="0.6096" layer="1"/>
 <wire x1="47.950684375" y1="52.395684375" x2="47.625" y2="52.07" width="0.6096" layer="1"/>
+<contactref element="C5" pad="1"/>
+<wire x1="48.39" y1="54.61" x2="48.39" y2="54.48" width="0.6096" layer="1"/>
+<wire x1="49.53" y1="52.629865625" x2="49.76418125" y2="52.395684375" width="0.6096" layer="1"/>
+<wire x1="48.39" y1="54.48" x2="49.025" y2="54.48" width="0.6096" layer="1"/>
+<wire x1="49.025" y1="54.48" x2="49.53" y2="53.975" width="0.6096" layer="1"/>
+<wire x1="49.53" y1="53.975" x2="49.53" y2="52.629865625" width="0.6096" layer="1"/>
+<wire x1="49.53" y1="52.629865625" x2="49.76418125" y2="52.395684375" width="0.6096" layer="1"/>
 </signal>
 <signal name="D+">
@@
 <wire x1="43.815" y1="53.975" x2="43.815" y2="52.2039375" width="0.6096" layer="16"/>
 <wire x1="43.815" y1="52.2039375" x2="51.5176125" y2="44.501325" width="0.6096" layer="16"/>
+<contactref element="C5" pad="2"/>
+<wire x1="45.59" y1="54.61" x2="44.45" y2="54.61" width="0.6096" layer="1"/>
+<wire x1="44.45" y1="54.61" x2="43.815" y2="53.975" width="0.6096" layer="1"/>
 </signal>
 <signal name="VCC">

Commit message: diode array
Parts:
- removed D1, D2, D3, D4, D5: (no value), fab:SOD123
- added U$2: INVERTER, SparkFun:SOT23-5
Connections:
- net D+: now also U$2.3; no longer D2.ANODE, D3.CATHODE
- net D-: now also U$2.4; no longer D1.ANODE, D4.CATHODE
- net GND: now also U$2.2
- net N$25: no longer D3.ANODE, D4.ANODE, D5.ANODE
- net VBUS: now also U$2.5; no longer D1.CATHODE, D2.CATHODE, D5.CATHODE
Routing:
- net N$25: track 44.7 -> 28.8 mm
- net GND: track 165.4 -> 175.9 mm, vias 9 -> 10
- net D-: track 38.6 -> 32.2 mm
- net VBUS: track 110.9 -> 107.0 mm
- net D+: track 38.9 -> 40.8 mm

Commit message: added power pins
Parts:
- added JP8, JP9: (no value), SparkFun:1X02
- moved JUMPER2 28.8 mm to (44.5, 31.8), turned to 180 degrees
Connections:
- net GND: now also JP8.1, JP9.1
- net VBUS: now also JP9.2
- net VCC: now also JP8.2
Routing:
- net GND: track 175.9 -> 218.0 mm, vias 10 -> 11
- net VCC: track 55.9 -> 71.6 mm
- net VBUS: track 107.0 -> 110.6 mm
- net RESET: track 179.9 -> 177.6 mm
- net N$9: track 28.7 -> 27.6 mm
- net N$10: track 26.6 -> 25.9 mm

Commit message: latest
Parts:
- added JP6: (no value), fab:2X03SMD
- moved C3 13.5 mm to (91.2, 57.0), turned to 90 degrees
- moved C4 1.73 mm to (101.7, 41.9), turned to 90 degrees
- moved S1 0.95 mm to (88.2, 49.7)
Connections:
- new net DAT: IC1.34, JP6.1
- net GND: now also JP6.6
- net RESET: now also JP6.5; no longer JP4.5
Routing:
- net RESET: track 177.6 -> 116.3 mm
- net DAT: track 0.00 -> 43.9 mm
- net GND: track 218.0 -> 246.9 mm, vias 11 -> 12
- net PE3: track 42.6 -> 36.0 mm
- net PE2: track 43.5 -> 38.5 mm
- net PE1: track 46.4 -> 42.0 mm
- net PE0: track 47.8 -> 45.3 mm
- net VBUS: track 110.6 -> 108.3 mm

Commit message: final pngs
Parts:
- removed C3: 0.1uF, fab:C1206
- removed JUMPER1, JUMPER2: 0, fab:R1206FAB
- added JUMPER: 0Ohm, fab:R1206FAB
- moved R2 6.37 mm to (43.7, 38.1), turned to 270 degrees
- moved JP9 5.08 mm to (47.0, 21.6), turned to 180 degrees
- moved U$2 1.62 mm to (90.5, 27.0)
- moved JP6 1.23 mm to (84.2, 60.5), turned to 180 degrees
Connections:
- net D+: now also IC1.27, JP3.1, U$2.4; no longer IC1.26, JP3.2, U$2.3
- net D-: now also IC1.26, JP3.2, U$2.3; no longer IC1.27, JP3.1, U$2.4
- net GND: no longer C3.2
- net RESET: no longer C3.1
- net VCC: now also JP6.2
Routing:
- net RESET: track 116.3 -> 33.4 mm
- net GND: track 246.9 -> 225.4 mm, vias 12 -> 9
- net VCC: track 71.6 -> 79.5 mm
- net D+: track 40.8 -> 34.1 mm
- net VBUS: track 108.3 -> 102.2 mm
- net D-: track 32.2 -> 38.2 mm
- net DAT: track 43.9 -> 47.5 mm
- net PA4: track 17.0 -> 14.6 mm
- net N$26: track 3.24 -> 2.13 mm
- net N$13: track 33.0 -> 32.4 mm
